Commit message: fixed ft_frame orientation

File: space_panda_description/urdf/space_panda.urdf_macro.xacro (robot description, xacro)
@@ -323,5 +323,5 @@
     <link name="${tf_prefix}ft_frame"/>
     <joint name="${tf_prefix}tool0-ft_frame" type="fixed">
-      <origin xyz="0 0 0.0" rpy="0 ${180*(pi/180)} ${-45*(pi/180)}"/>
+      <origin xyz="0 0 0.0" rpy="0 ${180*(pi/180)} ${45*(pi/180)}"/>
       <parent link="${tf_prefix}tool0"/>
       <child link="${tf_prefix}ft_frame"/>

Commit message: remove moveit dependencies and used robot state and model from franka directly

File: space_panda_description/urdf/space_panda.urdf_macro.xacro (robot description, xacro)
@@ -323,5 +323,5 @@
     <link name="${tf_prefix}ft_frame"/>
     <joint name="${tf_prefix}tool0-ft_frame" type="fixed">
-      <origin xyz="0 0 0.0" rpy="0 ${180*(pi/180)} ${45*(pi/180)}"/>
+      <origin xyz="0 0 0.0" rpy="0 ${0*(pi/180)} ${-90*(pi/180)}"/>
       <parent link="${tf_prefix}tool0"/>
       <child link="${tf_prefix}ft_frame"/>
